File: v1.1/Kicad/TRS80IJP_CPU.kicad_sch (KiCad schematic)
At the start: 18 parts

Commit message: Update Z32 label, Sync v1.1 Schematic to PCB
Parts:
- C40: footprint Capacitor_THT:CP_Radial_D4.0mm_P2.00mm -> TRS80:CP_Radial_D5.0mm_P2.50mm
- C70: footprint Capacitor_THT:CP_Radial_D6.3mm_P2.50mm -> TRS80:CP_Radial_D5.0mm_P2.50mm
Changed lines of the file:
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@@
       (effects (font (size 1.27 1.27)) (justify left))
     )
-    (property "Footprint" "Capacitor_THT:CP_Radial_D6.3mm_P2.50mm" (at 46.6852 162.56 0)
+    (property "Footprint" "TRS80:CP_Radial_D5.0mm_P2.50mm" (at 46.6852 162.56 0)
       (effects (font (size 1.27 1.27)) hide)
     )
@@
       (effects (font (size 1.27 1.27)) (justify left))
     )
-    (property "Footprint" "Capacitor_THT:CP_Radial_D4.0mm_P2.00mm" (at 61.9252 125.73 0)
-      (effects (font (size 1.27 1.27)) hide)
-    )
+    (property "Footprint" "TRS80:CP_Radial_D5.0mm_P2.50mm" (at 61.9252 125.73 0)
+      (effects (font (size 1.27 1.27)) hide)
+    )
