File: v1.1/Kicad/TRS80IJP_KEYBOARD.kicad_sch (KiCad schematic)
At the start: 4 parts, among them CN1 JP B KEYBOARD, CN2 KEYBOARD 2, CN3 US KEYBOARD

Commit message: Update Z32 label, Sync v1.1 Schematic to PCB
Parts:
- CN2: footprint Connector_PinHeader_2.54mm:PinHeader_1x09_P2.54mm_Vertical -> TRS80:CN2
Changed lines of the file:
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@@
       (effects (font (size 1.27 1.27)) (justify left))
     )
-    (property "Footprint" "Connector_PinHeader_2.54mm:PinHeader_1x09_P2.54mm_Vertical" (at 54.61 107.315 0)
+    (property "Footprint" "TRS80:CN2" (at 54.61 107.315 0)
       (effects (font (size 1.27 1.27)) hide)
     )
