File: v1.1/Kicad/TRS80IJP_POWER.kicad_sch (KiCad schematic)
At the start: 84 parts, among them J1 POWER, Q3 2SC1499, Q4 B531, Q5 2SA1015, Q6 B595

Commit message: Update Z32 label, Sync v1.1 Schematic to PCB
Parts:
- C12, C14, C6: footprint Capacitor_THT:CP_Radial_D5.0mm_P2.50mm -> TRS80:CP_Radial_D5.0mm_P2.50mm
- C5: footprint Capacitor_THT:CP_Radial_D10.0mm_P5.00mm -> TRS80:CP_Radial_P5.00mm
- C9: footprint Capacitor_THT:CP_Axial_L42.5mm_D20.0mm_P49.00mm_Horizontal -> TRS80:CP_Axial_L42.5mm_D20.0mm_P49.00mm
- CR3: footprint TRS80:Diode 3 10.16mm -> TRS80:Diode CR3
- Q3: footprint Package_TO_SOT_THT:TO-92_Inline -> TRS80:Q3
- Q4: footprint Package_TO_SOT_THT:TO-3 -> TRS80:Q4 TO-3
- Q5: footprint Package_TO_SOT_THT:TO-92_Inline -> TRS80:TO-92_Transistor
- Q6: footprint Package_TO_SOT_THT:TO-3 -> TRS80:Q6
- R17: footprint TRS80:Pot -> TRS80:Pot-R17
Changed lines of the file:
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@@
       (effects (font (size 1.27 1.27)) (justify left))
     )
-    (property "Footprint" "Capacitor_THT:CP_Radial_D10.0mm_P5.00mm" (at 190.8048 168.91 0)
+    (property "Footprint" "TRS80:CP_Radial_P5.00mm" (at 190.8048 168.91 0)
       (effects (font (size 1.27 1.27)) hide)
     )
@@
       (effects (font (size 1.27 1.27)) (justify left))
     )
-    (property "Footprint" "Package_TO_SOT_THT:TO-92_Inline" (at 196.85 133.985 0)
+    (property "Footprint" "TRS80:TO-92_Transistor" (at 196.85 133.985 0)
       (effects (font (size 1.27 1.27) italic) (justify left) hide)
     )
@@
       (effects (font (size 1.27 1.27)))
     )
-    (property "Footprint" "Capacitor_THT:CP_Radial_D5.0mm_P2.50mm" (at 211.1248 168.91 0)
+    (property "Footprint" "TRS80:CP_Radial_D5.0mm_P2.50mm" (at 211.1248 168.91 0)
       (effects (font (size 1.27 1.27)) hide)
     )
@@
       (effects (font (size 1.27 1.27)) (justify right))
     )
-    (property "Footprint" "TRS80:Diode 3 10.16mm" (at 237.49 172.72 0)
+    (property "Footprint" "TRS80:Diode CR3" (at 237.49 172.72 0)
       (effects (font (size 1.27 1.27)) hide)
     )
@@
       (effects (font (size 1.27 1.27)) (justify right))
     )
-    (property "Footprint" "TRS80:Pot" (at 113.03 143.51 0)
+    (property "Footprint" "TRS80:Pot-R17" (at 113.03 143.51 0)
       (effects (font (size 1.27 1.27)) hide)
     )
@@
       (effects (font (size 1.27 1.27)) (justify left))
     )
-    (property "Footprint" "Capacitor_THT:CP_Radial_D5.0mm_P2.50mm" (at 201.6252 129.54 0)
+    (property "Footprint" "TRS80:CP_Radial_D5.0mm_P2.50mm" (at 201.6252 129.54 0)
       (effects (font (size 1.27 1.27)) hide)
     )
@@
       (effects (font (size 1.27 1.27)) (justify left))
     )
-    (property "Footprint" "Capacitor_THT:CP_Axial_L42.5mm_D20.0mm_P49.00mm_Horizontal" (at 98.7552 67.31 0)
+    (property "Footprint" "TRS80:CP_Axial_L42.5mm_D20.0mm_P49.00mm" (at 98.7552 67.31 0)
       (effects (font (size 1.27 1.27)) hide)
     )
@@
       (effects (font (size 1.27 1.27)) (justify left))
     )
-    (property "Footprint" "Capacitor_THT:CP_Radial_D5.0mm_P2.50mm" (at 188.9252 55.88 0)
+    (property "Footprint" "TRS80:CP_Radial_D5.0mm_P2.50mm" (at 188.9252 55.88 0)
       (effects (font (size 1.27 1.27)) hide)
     )
@@
       (effects (font (size 1.27 1.27)))
     )
-    (property "Footprint" "Package_TO_SOT_THT:TO-3" (at 175.895 78.74 0)
+    (property "Footprint" "TRS80:Q4 TO-3" (at 175.895 78.74 0)
       (effects (font (size 1.27 1.27) italic) (justify left) hide)
     )
@@
       (effects (font (size 1.27 1.27)))
     )
-    (property "Footprint" "Package_TO_SOT_THT:TO-92_Inline" (at 184.785 86.36 0)
+    (property "Footprint" "TRS80:Q3" (at 184.785 86.36 0)
       (effects (font (size 1.27 1.27) italic) (justify left) hide)
     )
@@
       (effects (font (size 1.27 1.27)))
     )
-    (property "Footprint" "Package_TO_SOT_THT:TO-3" (at 140.335 30.48 0)
+    (property "Footprint" "TRS80:Q6" (at 140.335 30.48 0)
       (effects (font (size 1.27 1.27) italic) (justify left) hide)
     )
