File: v1.1/Kicad/TRS80IJP_TAPE.kicad_sch (KiCad schematic)
At the start: 43 parts, among them J3 CASS OUT, K1 5V Relay

Commit message: Update Z32 label, Sync v1.1 Schematic to PCB
Parts:
- C1: footprint Capacitor_THT:CP_Radial_D5.0mm_P2.50mm -> TRS80:CP_Radial_D5.0mm_P2.50mm
- C19: footprint Capacitor_THT:CP_Radial_D8.0mm_P5.00mm -> TRS80:CP_Radial_P5.00mm
- CR4: footprint Diode_THT:D_DO-41_SOD81_P10.16mm_Horizontal -> TRS80:Diode 10.16mm
Changed lines of the file:
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@@
       (effects (font (size 1.27 1.27)) (justify left))
     )
-    (property "Footprint" "Capacitor_THT:CP_Radial_D8.0mm_P5.00mm" (at 306.07 245.4148 0)
+    (property "Footprint" "TRS80:CP_Radial_P5.00mm" (at 306.07 245.4148 0)
       (effects (font (size 1.27 1.27)) hide)
     )
@@
       (effects (font (size 1.27 1.27)) (justify left))
     )
-    (property "Footprint" "Diode_THT:D_DO-41_SOD81_P10.16mm_Horizontal" (at 292.1 177.8 0)
+    (property "Footprint" "TRS80:Diode 10.16mm" (at 292.1 177.8 0)
       (effects (font (size 1.27 1.27)) hide)
     )
@@
       (effects (font (size 1.27 1.27)) (justify left))
     )
-    (property "Footprint" "Capacitor_THT:CP_Radial_D5.0mm_P2.50mm" (at 106.3752 110.49 0)
-      (effects (font (size 1.27 1.27)) hide)
-    )
+    (property "Footprint" "TRS80:CP_Radial_D5.0mm_P2.50mm" (at 106.3752 110.49 0)
+      (effects (font (size 1.27 1.27)) hide)
+    )
