File: v1.1/Kicad/TRS80IJP_VIDEO.kicad_sch (KiCad schematic)
At the start: 38 parts, among them J2 VIDEO OUT, Q1 2SC1815, Q2 2SA1015

Commit message: Update Z32 label, Sync v1.1 Schematic to PCB
Parts:
- C4: footprint Capacitor_THT:CP_Radial_D5.0mm_P2.50mm -> TRS80:CP_Radial_D5.0mm_P2.50mm
- Q1, Q2: footprint Package_TO_SOT_THT:TO-92_Inline -> TRS80:TO-92_Transistor
Changed lines of the file:
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@@
       (effects (font (size 1.27 1.27)) (justify left))
     )
-    (property "Footprint" "Package_TO_SOT_THT:TO-92_Inline" (at 363.22 225.425 0)
+    (property "Footprint" "TRS80:TO-92_Transistor" (at 363.22 225.425 0)
       (effects (font (size 1.27 1.27) italic) (justify left) hide)
     )
@@
       (effects (font (size 1.27 1.27)) (justify left))
     )
-    (property "Footprint" "Package_TO_SOT_THT:TO-92_Inline" (at 349.25 189.865 0)
+    (property "Footprint" "TRS80:TO-92_Transistor" (at 349.25 189.865 0)
       (effects (font (size 1.27 1.27) italic) (justify left) hide)
     )
@@
       (effects (font (size 1.27 1.27)) (justify left))
     )
-    (property "Footprint" "Capacitor_THT:CP_Radial_D5.0mm_P2.50mm" (at 390.8552 243.84 0)
-      (effects (font (size 1.27 1.27)) hide)
-    )
+    (property "Footprint" "TRS80:CP_Radial_D5.0mm_P2.50mm" (at 390.8552 243.84 0)
+      (effects (font (size 1.27 1.27)) hide)
+    )
